File: pcb/Signal Generator.kicad_sch (KiCad schematic)
At the start: 7 parts, among them J1 AudioJack3, J2 Conn_02x02_Odd_Even, J3 Screw_Terminal_01x04, J4 MEM2080-00-128-00-A

Commit message: Updated PCB
Parts:
- J1: footprint Signal Generator Components:SJ-3523-SMT-TR-1 -> Signal Generator Components:SJ-3523-SMT-TR
Connections:
- net GND: now also J2.2 (Pin_2), J2.4 (Pin_4); no longer J2.1 (Pin_1), J2.3 (Pin_3)
- net Output Stage/CH1_OUT: now also J2.1 (Pin_1); no longer J2.2 (Pin_2)
- net Output Stage/CH2_OUT: now also J2.3 (Pin_3); no longer J2.4 (Pin_4)
Other:
- moved on the sheet: J2
Changed lines of the file:
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@@
       (effects (font (size 1.27 1.27)) (justify right))
     )
-    (property "Footprint" "Signal Generator Components:SJ-3523-SMT-TR-1" (at 185.42 52.07 0)
+    (property "Footprint" "Signal Generator Components:SJ-3523-SMT-TR" (at 185.42 52.07 0)
       (effects (font (size 1.27 1.27)) hide)
     )
@@
     )
   )
-  (symbol (lib_id "Connector_Generic:Conn_02x02_Odd_Even") (at 187.96 81.28 180) (unit 1)
+  (symbol (lib_id "Connector_Generic:Conn_02x02_Odd_Even") (at 185.42 81.28 0) (mirror x) (unit 1)
     (in_bom yes) (on_board yes) (dnp no)
     (property "Reference" "J2" (at 196.85 78.74 0)
-      (effects (font (size 1.27 1.27)) (justify right))
+      (effects (font (size 1.27 1.27)) (justify left))
     )
     (property "Value" "Conn_02x02_Odd_Even" (at 196.85 81.28 0)
-      (effects (font (size 1.27 1.27)) (justify right))
+      (effects (font (size 1.27 1.27)) (justify left))
     )
-    (property "Footprint" "Connector_PinHeader_2.54mm:PinHeader_2x02_P2.54mm_Horizontal" (at 187.96 81.28 0)
+    (property "Footprint" "Connector_PinHeader_2.54mm:PinHeader_2x02_P2.54mm_Horizontal" (at 185.42 81.28 0)
       (effects (font (size 1.27 1.27)) hide)
     )
-    (property "Datasheet" "~" (at 187.96 81.28 0)
+    (property "Datasheet" "~" (at 185.42 81.28 0)
       (effects (font (size 1.27 1.27)) hide)
     )
-    (property "PN" "10129382-904001BLF" (at 187.96 81.28 0)
+    (property "PN" "10129382-904001BLF" (at 185.42 81.28 0)
       (effects (font (size 1.27 1.27)) hide)
     )
