File: pcb/MCU.kicad_sch (KiCad schematic)
At the start: 16 parts, among them J6 Conn_01x04, SW1 SW_Push, SW1 SW_SPDT, U3 STM32F103RBTx, Y1 TG2520SMN_16.0000M-MCGNNM0

Commit message: Updated PCB to correct some connection errors
Connections:
- net DAC1: now also U3.20 (PA4); no longer U3.21 (PA5)
- net DAC2: now also U3.21 (PA5); no longer U3.22 (PA6)
- net OSC: now also U3.5 (PD0); no longer U3.25 (PC5)
- net SD_Detect: now also U3.61 (PB8); no longer U3.58 (PB6)
- net SWCLK: now also J6.3 (Pin_3), U3.49 (PA14); no longer J6.2 (Pin_2), U3.35 (PB14)
- net SWDIO: now also J6.2 (Pin_2), U3.46 (PA13); no longer J6.3 (Pin_3), U3.34 (PB13)
- net UART1_RX: now also U3.59 (PB7); no longer U3.61 (PB8)
- net UART1_TX: now also U3.58 (PB6); no longer U3.59 (PB7)
- no-connect marks 37 -> 35
Changed lines of the file:
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@@
-(kicad_sch (version 20221206) (generator eeschema)
+(kicad_sch (version 20230121) (generator eeschema)
   (paper "A4")
   (title_block
@@
   )
   (no_connect (at 111.76 91.44))
-  (no_connect (at 111.76 93.98))
   (no_connect (at 111.76 81.28))
   (no_connect (at 111.76 60.96))
-  (no_connect (at 76.2 78.74))
+  (no_connect (at 76.2 93.98))
   (no_connect (at 76.2 86.36))
+  (no_connect (at 76.2 81.28))
   (no_connect (at 76.2 119.38))
   (no_connect (at 111.76 106.68))
-  (no_connect (at 76.2 121.92))
   (no_connect (at 111.76 78.74))
   (no_connect (at 76.2 114.3))
@@
   (no_connect (at 76.2 91.44))
   (no_connect (at 111.76 88.9))
+  (no_connect (at 76.2 76.2))
   (no_connect (at 76.2 99.06))
   (no_connect (at 76.2 88.9))
   (no_connect (at 111.76 132.08))
-  (no_connect (at 111.76 71.12))
   (no_connect (at 111.76 83.82))
   (no_connect (at 111.76 104.14))
   (no_connect (at 111.76 68.58))
   (no_connect (at 76.2 104.14))
+  (no_connect (at 111.76 76.2))
   (no_connect (at 76.2 111.76))
   (no_connect (at 111.76 109.22))
@@
   (no_connect (at 111.76 127))
   (no_connect (at 76.2 109.22))
-  (no_connect (at 111.76 96.52))
   (no_connect (at 177.8 129.54))
   (no_connect (at 76.2 106.68))
   (no_connect (at 76.2 83.82))
-  (no_connect (at 76.2 71.12))
   (no_connect (at 76.2 101.6))
   (wire (pts (xy 181.61 67.31) (xy 193.04 67.31))
@@
     (stroke (width 0) (type default))
   )
+  (wire (pts (xy 74.93 71.12) (xy 76.2 71.12))
+    (stroke (width 0) (type default))
+  )
   (wire (pts (xy 151.13 92.71) (xy 151.13 95.25))
     (stroke (width 0) (type default))
@@
     (stroke (width 0) (type default))
   )
+  (wire (pts (xy 113.03 96.52) (xy 111.76 96.52))
+    (stroke (width 0) (type default))
+  )
   (wire (pts (xy 223.52 99.06) (xy 223.52 101.6))
     (stroke (width 0) (type default))
@@
     (stroke (width 0) (type default))
   )
-  (wire (pts (xy 113.03 76.2) (xy 111.76 76.2))
-    (stroke (width 0) (type default))
-  )
   (wire (pts (xy 193.04 67.31) (xy 204.47 67.31))
     (stroke (width 0) (type default))
@@
     (stroke (width 0) (type default))
   )
+  (wire (pts (xy 111.76 71.12) (xy 113.03 71.12))
+    (stroke (width 0) (type default))
+  )
   (wire (pts (xy 113.03 99.06) (xy 111.76 99.06))
     (stroke (width 0) (type default))
@@
     (stroke (width 0) (type default))
   )
-  (wire (pts (xy 74.93 93.98) (xy 76.2 93.98))
-    (stroke (width 0) (type default))
-  )
   (wire (pts (xy 193.04 57.15) (xy 204.47 57.15))
     (stroke (width 0) (type default))
@@
     (stroke (width 0) (type default))
   )
-  (wire (pts (xy 113.03 139.7) (xy 111.76 139.7))
-    (stroke (width 0) (type default))
-  )
   (wire (pts (xy 113.03 142.24) (xy 111.76 142.24))
     (stroke (width 0) (type default))
   )
+  (wire (pts (xy 113.03 93.98) (xy 111.76 93.98))
+    (stroke (width 0) (type default))
+  )
   (wire (pts (xy 151.13 95.25) (xy 153.67 95.25))
     (stroke (width 0) (type default))
@@
     (stroke (width 0) (type default))
   )
-  (wire (pts (xy 113.03 137.16) (xy 111.76 137.16))
-    (stroke (width 0) (type default))
-  )
   (polyline (pts (xy 199.39 116.84) (xy 199.39 143.51))
     (stroke (width 0) (type default))
@@
     (effects (font (size 1.27 1.27)) (justify left bottom))
   )
-  (label "OSC" (at 74.93 93.98 180) (fields_autoplaced)
-    (effects (font (size 1.27 1.27)) (justify right bottom))
-  )
   (label "NRST" (at 161.29 152.4 180) (fields_autoplaced)
     (effects (font (size 1.27 1.27)) (justify right bottom))
   )
-  (label "SWCLK" (at 113.03 139.7 0) (fields_autoplaced)
-    (effects (font (size 1.27 1.27)) (justify left bottom))
-  )
-  (label "SWCLK" (at 161.29 154.94 180) (fields_autoplaced)
+  (label "SWDIO" (at 113.03 93.98 0) (fields_autoplaced)
+    (effects (font (size 1.27 1.27)) (justify left bottom))
+  )
+  (label "SWCLK" (at 161.29 157.48 180) (fields_autoplaced)
+    (effects (font (size 1.27 1.27)) (justify right bottom))
+  )
+  (label "OSC" (at 74.93 71.12 180) (fields_autoplaced)
     (effects (font (size 1.27 1.27)) (justify right bottom))
   )
@@
     (effects (font (size 1.27 1.27)) (justify left bottom))
   )
-  (label "SWDIO" (at 113.03 137.16 0) (fields_autoplaced)
+  (label "SWCLK" (at 113.03 96.52 0) (fields_autoplaced)
     (effects (font (size 1.27 1.27)) (justify left bottom))
   )
@@
     (effects (font (size 1.27 1.27)) (justify right bottom))
   )
-  (label "SWDIO" (at 161.29 157.48 180) (fields_autoplaced)
+  (label "SWDIO" (at 161.29 154.94 180) (fields_autoplaced)
     (effects (font (size 1.27 1.27)) (justify right bottom))
   )
@@
     (effects (font (size 1.27 1.27)) (justify right bottom))
   )
-  (hierarchical_label "UART1_TX" (shape output) (at 113.03 121.92 0) (fields_autoplaced)
-    (effects (font (size 1.27 1.27)) (justify left))
-  )
   (hierarchical_label "SPI1_SCK" (shape output) (at 113.03 111.76 0) (fields_autoplaced)
     (effects (font (size 1.27 1.27)) (justify left))
@@
     (effects (font (size 1.27 1.27)) (justify left))
   )
+  (hierarchical_label "DAC2" (shape output) (at 113.03 73.66 0) (fields_autoplaced)
+    (effects (font (size 1.27 1.27)) (justify left))
+  )
+  (hierarchical_label "UART1_RX" (shape output) (at 113.03 121.92 0) (fields_autoplaced)
+    (effects (font (size 1.27 1.27)) (justify left))
+  )
   (hierarchical_label "ADC2" (shape input) (at 113.03 66.04 0) (fields_autoplaced)
     (effects (font (size 1.27 1.27)) (justify left))
   )
-  (hierarchical_label "SD_Detect" (shape input) (at 113.03 119.38 0) (fields_autoplaced)
+  (hierarchical_label "UART1_TX" (shape output) (at 113.03 119.38 0) (fields_autoplaced)
     (effects (font (size 1.27 1.27)) (justify left))
   )
@@
     (effects (font (size 1.27 1.27)) (justify left))
   )
+  (hierarchical_label "SD_Detect" (shape input) (at 113.03 124.46 0) (fields_autoplaced)
+    (effects (font (size 1.27 1.27)) (justify left))
+  )
   (hierarchical_label "SPI1_MISO" (shape input) (at 113.03 114.3 0) (fields_autoplaced)
     (effects (font (size 1.27 1.27)) (justify left))
@@
     (effects (font (size 1.27 1.27)) (justify left))
   )
-  (hierarchical_label "DAC2" (shape output) (at 113.03 76.2 0) (fields_autoplaced)
-    (effects (font (size 1.27 1.27)) (justify left))
-  )
-  (hierarchical_label "DAC1" (shape output) (at 113.03 73.66 0) (fields_autoplaced)
-    (effects (font (size 1.27 1.27)) (justify left))
-  )
-  (hierarchical_label "UART1_RX" (shape output) (at 113.03 124.46 0) (fields_autoplaced)
-    (effects (font (size 1.27 1.27)) (justify left))
-  )
+  (hierarchical_label "DAC1" (shape output) (at 113.03 71.12 0) (fields_autoplaced)
+    (effects (font (size 1.27 1.27)) (justify left))
+  )

Commit message: Fixed FTDI connection to the stm32
Connections:
- no-connect marks 35 -> 37
Changed lines of the file:
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@@
   (no_connect (at 111.76 81.28))
   (no_connect (at 111.76 60.96))
+  (no_connect (at 111.76 137.16))
   (no_connect (at 76.2 93.98))
+  (no_connect (at 111.76 139.7))
   (no_connect (at 76.2 86.36))
   (no_connect (at 76.2 81.28))
