File: pcb/MCU.kicad_sch (KiCad schematic)
At the start: 16 parts, among them J6 Conn_01x04, SW1 SW_Push, SW1 SW_SPDT, U3 STM32F103RBTx, Y1 TG2520SMN_16.0000M-MCGNNM0

Commit message: Switch to stm32f205
Parts:
- removed C?: 10n, Capacitor_SMD:C_0603_1608Metric, symbol Device:C
- removed U3: STM32F103RBTx, Package_QFP:LQFP-64_10x10mm_P0.5mm, symbol MCU_ST_STM32F1:STM32F103RBTx
- removed Y1: TG2520SMN_16.0000M-MCGNNM0, Signal Generator Components:TG2520SMN_16.0000M-MCGNNM0, symbol Signal Generator Components:TG2520SMN_16.0000M-MCGNNM0
- added C? (x2): 100n, Capacitor_SMD:C_0603_1608Metric, symbol Device:C
- added C? (x2): 2.2u, Capacitor_SMD:C_0603_1608Metric, symbol Device:C
- added U3: STM32F205RCTx, Package_QFP:LQFP-64_10x10mm_P0.5mm, symbol MCU_ST_STM32F2:STM32F205RCTx
- added U4: FT5HN, Oscillator:Oscillator_SMD_Fox_FT5H_5.0x3.2mm, symbol Oscillator:FT5HN
Connections:
- net +3.3V: now also C?.1, C?.1, U3.1 (VBAT), U3.13 (VDDA), U3.19 (VDD), U3.32 (VDD), U3.48 (VDD), U3.64 (VDD), U4.4 (VDD)
- net ADC1: now also U3.15 (PA1)
- net ADC2: now also U3.16 (PA2)
- net BOOT0: now also U3.60 (BOOT0)
- net DAC1: now also U3.20 (PA4)
- net DAC2: now also U3.21 (PA5)
- net GND: now also C?.2, C?.2, C?.2, C?.2, U3.12 (VSSA), U3.18 (VSS), U3.63 (VSS), U4.1 (GND), U4.2 (GND)
- net LED_DIN: now also U3.36 (PB15)
- net NRST: now also U3.7 (NRST)
- net OSC: now also U3.5 (PH0), U4.3 (OUT)
- net SD_Detect: now also U3.61 (PB8)
- net SWCLK: now also U3.49 (PA14)
- net SWDIO: now also U3.46 (PA13)
- net UART1_RX: now also U3.43 (PA10)
- net UART1_TX: now also U3.42 (PA9)
- new net: C?.1, U3.47 (VCAP_2)
- new net: C?.1, U3.31 (VCAP_1)
- new net SD_CMD: U3.54 (PD2)
- new net SD_D0: U3.39 (PC8)
- new net SD_D1: U3.40 (PC9)
- new net SD_D2: U3.51 (PC10)
- new net SD_D3: U3.52 (PC11)
- new net SD_SCK: U3.53 (PC12)
- no-connect marks 37 -> 35
Other:
- note added: "Oscillator (25MHz)"
- note removed: "Oscillator"
- moved on the sheet: C?, D3, J6, R17

Commit message: Prepared PCB rev 3
Parts:
- J6: footprint Connector_PinHeader_2.54mm:PinHeader_1x04_P2.54mm_Horizontal -> Connector_PinHeader_2.54mm:PinHeader_1x04_P2.54mm_Vertical
Changed lines of the file:
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@@
       (effects (font (size 1.27 1.27)) (justify left))
     )
-    (property "Footprint" "Connector_PinHeader_2.54mm:PinHeader_1x04_P2.54mm_Horizontal" (at 167.64 160.02 0)
+    (property "Footprint" "Connector_PinHeader_2.54mm:PinHeader_1x04_P2.54mm_Vertical" (at 167.64 160.02 0)
       (effects (font (size 1.27 1.27)) hide)
     )
