File: pcb/Signal Generator.kicad_pcb (KiCad board)
At the start: 4 copper layers, 36 x 60 mm, 67 parts, among them J1 AudioJack3, J2 Conn_02x02_Odd_Even, J3 Screw_Terminal_01x04, J4 MEM2080-00-128-00-A, J5 USB_C_Receptacle_USB2.0, J6 Conn_01x04, SW1 SW_Push, SW2 SW_SPDT, U1 FT230XQ, U2 Opamp_Dual, U3 STM32F103RBTx, U4 LD39050PU33R, U5 TLV61048, U6 LDK320AM120R, Y1 TG2520SMN_16.0000M-MCGNNM0

Commit message: Switch to stm32f205
Parts:
- removed the C19 at (99.2, 124.8)
- removed Y1: TG2520SMN_16.0000M-MCGNNM0, Signal Generator Components:TG2520SMN_16.0000M-MCGNNM0
- added C15: 2.2u, Capacitor_SMD:C_0603_1608Metric, F.Cu at (113.5, 117.3)
- added C20: 100n, Capacitor_SMD:C_0603_1608Metric, F.Cu at (99.3, 124.8)
- added C21: 100n, Capacitor_SMD:C_0603_1608Metric, F.Cu at (100.5, 117.3)
- added C22: 1u, Capacitor_SMD:C_0603_1608Metric, F.Cu at (99.3, 121.2)
- added U4: FT5HN, Oscillator:Oscillator_SMD_Fox_FT5H_5.0x3.2mm, F.Cu at (95.2, 122.8)
- C14: value 10n -> 2.2u
- U3: value STM32F103RBTx -> STM32F205RCTx
- moved C14 12.4 mm to (107.7, 130.6), turned to 180 degrees
- moved C3 4.61 mm to (92.5, 129.8), turned to -90 degrees
- moved C1 3.55 mm to (93.2, 127.0)
- moved C17 1.25 mm to (102.0, 116.2), turned to 90 degrees
- moved C18 1.25 mm to (112.0, 116.2), turned to 90 degrees
- renumbered C2 to C1, C9 to C10, C10 to C11, C11 to C12, C12 to C13, C15 to C16, C16 to C17, C17 to C18, C18 to C19, C1 to C2, C22 to C23, C20 to C24, C23 to C26, C24 to C27, C26 to C28, C28 to C29, C27 to C30, C8 to C7, C13 to C8, C7 to C9, R5 to R1, R15 to R10, R7 to R11, R9 to R13, R11 to R14, R14 to R15, R6 to R2, R1 to R3, R2 to R4, R3 to R5, R4 to R6, R8 to R7, R10 to R8, R13 to R9, U4 to U5, U5 to U6, U6 to U7
Connections:
- C14 pad 1: +3.3V -> Net-(U3-VCAP_1)
- J4 pad P1: unconnected-(J4-DAT2-PadP1) -> /SD_D2
- J4 pad P2: /SD_CS -> /SD_D3
- J4 pad P3: /SD_MOSI -> /SD_CMD
- J4 pad P7: /SD_MISO -> /SD_D0
- J4 pad P8: unconnected-(J4-DAT1-PadP8) -> /SD_D1
- U3 pad 31: GND -> Net-(U3-VCAP_1)
- U3 pad 39: unconnected-(U3-PC8-Pad39) -> /SD_D0
- U3 pad 40: unconnected-(U3-PC9-Pad40) -> /SD_D1
- U3 pad 42: unconnected-(U3-PA9-Pad42) -> /MCU/UART1_TX
- U3 pad 43: unconnected-(U3-PA10-Pad43) -> /MCU/UART1_RX
- U3 pad 47: GND -> Net-(U3-VCAP_2)
- U3 pad 50: /SD_CS -> unconnected-(U3-PA15-Pad50)
- U3 pad 51: unconnected-(U3-PC10-Pad51) -> /SD_D2
- U3 pad 52: unconnected-(U3-PC11-Pad52) -> /SD_D3
- U3 pad 53: unconnected-(U3-PC12-Pad53) -> /SD_SCK
- U3 pad 54: unconnected-(U3-PD2-Pad54) -> /SD_CMD
- U3 pad 55: /SD_SCK -> unconnected-(U3-PB3-Pad55)
- U3 pad 56: /SD_MISO -> unconnected-(U3-PB4-Pad56)
- U3 pad 57: /SD_MOSI -> unconnected-(U3-PB5-Pad57)
- U3 pad 58: /MCU/UART1_TX -> unconnected-(U3-PB6-Pad58)
- U3 pad 59: /MCU/UART1_RX -> unconnected-(U3-PB7-Pad59)
Routing:
- net /SD_MISO: track 26.7 -> 0.00 mm, vias 1 -> 0
- net /SD_D1: track 0.00 -> 25.9 mm, vias 0 -> 2
- net /SD_D3: track 0.00 -> 25.1 mm, vias 0 -> 2
- net /SD_CMD: track 0.00 -> 24.7 mm, vias 0 -> 1
- net /SD_D0: track 0.00 -> 24.4 mm, vias 0 -> 2
- net /SD_D2: track 0.00 -> 24.2 mm, vias 0 -> 2
- net /SD_MOSI: track 24.1 -> 0.00 mm, vias 1 -> 0
- net /SD_CS: track 22.9 -> 0.00 mm, vias 2 -> 0
- net /MCU/UART1_RX: track 3.78 -> 16.0 mm
- net /MCU/UART1_TX: track 7.64 -> 15.9 mm
- net +3.3V: track 37.1 -> 33.4 mm
- net Net-(U3-VCAP_1): track 0.00 -> 3.06 mm
- net Net-(U3-VCAP_2): track 0.00 -> 2.74 mm
- net /ADC2: track 19.2 -> 20.7 mm
- net +12VA: track 53.7 -> 52.9 mm
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Other:
- board text added: "Rev 3"
- board text removed: "Rev 2"

Commit message: Prepared PCB rev 3
Parts:
- J6: footprint Connector_PinHeader_2.54mm:PinHeader_1x04_P2.54mm_Horizontal -> Connector_PinHeader_2.54mm:PinHeader_1x04_P2.54mm_Vertical
- moved R17 4.26 mm to (116.8, 127.0), turned to -45 degrees
Routing:
- net /MCU/LED_DIN: track 9.14 -> 4.06 mm
- net Net-(D3-DIN): track 12.8 -> 9.98 mm
