File: pcb/Signal Generator.kicad_pcb (KiCad board)
At the start: 4 copper layers, 36 x 60 mm, 70 parts, among them J1 AudioJack3, J2 Conn_02x02_Odd_Even, J3 Screw_Terminal_01x04, J4 MEM2080-00-128-00-A, J5 USB_C_Receptacle_USB2.0, J6 Conn_01x04, SW1 SW_Push, SW2 SW_SPDT, U1 FT230XQ, U2 Opamp_Dual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

Commit message: Updated pbc library paths
Parts:
- J6: moved to F.Cu
- turned J6 to -90 degrees
Changed lines of the file:
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@@
     (pad "6" smd roundrect (at 1.3 -0.95 180) (size 0.6 1.1) (layers "F.Cu" "F.Paste" "F.Mask") (roundrect_rratio 0.08333333333)
       (net 3 "GND") (pinfunction "FREQ") (pintype "input"))
-    (model "${SIGNAL_GENERATOR}/pcb-library/3D Models/TLV61048DBVT.step"
+    (model "${SIGNAL_GENERATOR}/3D Models/TLV61048DBVT.step"
       (offset (xyz 0 0 0))
       (scale (xyz 1 1 1))
@@
     (pad "2" smd rect (at 1.185 0 270) (size 0.98 3.4) (layers "F.Cu" "F.Paste" "F.Mask")
       (net 36 "Net-(D4-A)") (pinfunction "2") (pintype "passive") (thermal_bridge_angle 45))
-    (model ":SIGNAL_GENERATOR:pcb-library/3D Models/XAL4030.step"
+    (model "${SIGNAL_GENERATOR}/3D Models/XAL4030.step"
       (offset (xyz 0 0 0.05))
       (scale (xyz 1 1 1))
@@
     )
   )
+  (footprint "Connector_PinHeader_2.54mm:PinHeader_1x04_P2.54mm_Vertical" (layer "F.Cu")
+    (at 124.04 107.5 -90)
+    (descr "Through hole straight pin header, 1x04, 2.54mm pitch, single row")
+    (tags "Through hole pin header THT 1x04 2.54mm single row")
+    (property "Sheetfile" "MCU.kicad_sch")
+    (property "Sheetname" "MCU")
+    (property "ki_description" "Generic connector, single row, 01x04, script generated (kicad-library-utils/schlib/autogen/connector/)")
+    (property "ki_keywords" "connector")
+    (attr through_hole)
+    (fp_text reference "J6" (at 0 -2.33 90) (layer "F.SilkS") hide
+        (effects (font (size 1 1) (thickness 0.15)))
+    )
+    (fp_text value "Conn_01x04" (at 0 9.95 90) (layer "F.Fab") hide
+        (effects (font (size 1 1) (thickness 0.15)))
+    )
+    (fp_text user "${REFERENCE}" (at 0 3.81) (layer "F.Fab")
+        (effects (font (size 1 1) (thickness 0.15)))
+    )
+    (fp_line (start -1.8 -1.8) (end -1.8 9.4)
+      (stroke (width 0.05) (type solid)) (layer "F.CrtYd"))
+    (fp_line (start -1.8 9.4) (end 1.8 9.4)
+      (stroke (width 0.05) (type solid)) (layer "F.CrtYd"))
+    (fp_line (start 1.8 -1.8) (end -1.8 -1.8)
+      (stroke (width 0.05) (type solid)) (layer "F.CrtYd"))
+    (fp_line (start 1.8 9.4) (end 1.8 -1.8)
+      (stroke (width 0.05) (type solid)) (layer "F.CrtYd"))
+    (fp_line (start -1.27 -0.635) (end -0.635 -1.27)
+      (stroke (width 0.1) (type solid)) (layer "F.Fab"))
+    (fp_line (start -1.27 8.89) (end -1.27 -0.635)
+      (stroke (width 0.1) (type solid)) (layer "F.Fab"))
+    (fp_line (start -0.635 -1.27) (end 1.27 -1.27)
+      (stroke (width 0.1) (type solid)) (layer "F.Fab"))
+    (fp_line (start 1.27 -1.27) (end 1.27 8.89)
+      (stroke (width 0.1) (type solid)) (layer "F.Fab"))
+    (fp_line (start 1.27 8.89) (end -1.27 8.89)
+      (stroke (width 0.1) (type solid)) (layer "F.Fab"))
+    (pad "1" thru_hole rect (at 0 0 270) (size 1.7 1.7) (drill 1) (layers "*.Cu" "*.Mask")
+      (net 59 "/MCU/NRST") (pinfunction "Pin_1") (pintype "passive"))
+    (pad "2" thru_hole oval (at 0 2.54 270) (size 1.7 1.7) (drill 1) (layers "*.Cu" "*.Mask")
+      (net 46 "/MCU/SWDIO") (pinfunction "Pin_2") (pintype "passive"))
+    (pad "3" thru_hole oval (at 0 5.08 270) (size 1.7 1.7) (drill 1) (layers "*.Cu" "*.Mask")
+      (net 37 "/MCU/SWCLK") (pinfunction "Pin_3") (pintype "passive"))
+    (pad "4" thru_hole oval (at 0 7.62 270) (size 1.7 1.7) (drill 1) (layers "*.Cu" "*.Mask")
+      (net 3 "GND") (pinfunction "Pin_4") (pintype "passive"))
+    (model "${KICAD6_3DMODEL_DIR}/Connector_PinHeader_2.54mm.3dshapes/PinHeader_1x04_P2.54mm_Vertical.wrl"
+      (offset (xyz 0 0 0))
+      (scale (xyz 1 1 1))
+      (rotate (xyz 0 0 0))
+    )
+  )
   (footprint "Resistor_SMD:R_0603_1608Metric" (layer "F.Cu")
     (at 106 108 -90)
@@
     (pad "S1" thru_hole oval (at 4.32 0 180) (size 1 1.8) (drill oval 0.6 1.4) (layers "*.Cu" "*.Mask")
       (net 3 "GND") (pinfunction "SHIELD") (pintype "passive"))
-    (model "${SIGNAL_GENERATOR}/pcb-library/3D Models/USB4105-GF-A.step"
+    (model "${SIGNAL_GENERATOR}/3D Models/USB4105-GF-A.step"
       (offset (xyz 0 0 0))
       (scale (xyz 1 1 1))
@@
     (pad "2" smd rect (at 3.35 0 180) (size 2.05 3.8) (layers "F.Cu" "F.Paste" "F.Mask")
       (net 3 "GND") (pintype "passive"))
-    (model ":SIGNAL_GENERATOR:pcb-library/3D Models/WCAP-PSHP.step"
+    (model "${SIGNAL_GENERATOR}/3D Models/WCAP-PSHP.step"
       (offset (xyz 0 0 0))
       (scale (xyz 1 1 1))
@@
     (pad "5" smd rect (at 1.15 -0.95) (size 0.6 1.2) (layers "F.Cu" "F.Paste" "F.Mask")
       (net 58 "+12VA") (pinfunction "OUT") (pintype "power_out"))
-    (model "${SIGNAL_GENERATOR}/pcb-library/3D Models/LDK320AM120R.step"
+    (model "${SIGNAL_GENERATOR}/3D Models/LDK320AM120R.step"
       (offset (xyz 0 0 0))
       (scale (xyz 1 1 1))
@@
     (pad "T" smd rect (at 11.8 3.8 180) (size 2.6 2.8) (layers "F.Cu" "F.Paste" "F.Mask")
       (net 57 "/Output Stage/CH2_OUT") (pintype "passive"))
-    (model ":SIGNAL_GENERATOR:pcb-library/3D Models/SJ-3523-SMT-TR.stp"
+    (model "${SIGNAL_GENERATOR}/3D Models/SJ-3523-SMT-TR.stp"
       (offset (xyz 7.35 0 2.55))
       (scale (xyz 1 1 1))
@@
     (pad "7" smd rect (at 0 0) (size 1.75 2.5) (layers "F.Cu" "F.Paste" "F.Mask")
       (net 3 "GND") (pinfunction "PAD") (pintype "power_in"))
-    (model "${SIGNAL_GENERATOR}/pcb-library/3D Models/LD39050PU33R.step"
+    (model "${SIGNAL_GENERATOR}/3D Models/LD39050PU33R.step"
       (offset (xyz 0 0 0))
       (scale (xyz 1 1 1))
@@
     (pad "4" smd rect (at 2.2 -1.6) (size 1.6 1.1) (layers "F.Cu" "F.Paste" "F.Mask")
       (net 9 "unconnected-(D3-DO-Pad4)") (pinfunction "DO") (pintype "output+no_connect"))
-    (model "${KICAD6_3DMODEL_DIR}/LED_SMD.3dshapes/LED_Inolux_IN-PI554FCH_PLCC4_5.0x5.0mm_P3.2mm.wrl"
+    (model "${SIGNAL_GENERATOR}/3D Models/IN-PI55QA.step"
       (offset (xyz 0 0 0))
       (scale (xyz 1 1 1))
-      (rotate (xyz 0 0 0))
+      (rotate (xyz -90 0 0))
     )
   )
@@
     (pad "3" thru_hole circle (at 6 5.5) (size 1.524 1.524) (drill 0.762) (layers "*.Cu" "*.Mask")
       (net 12 "+3.3V") (pinfunction "C") (pintype "passive"))
-    (model ":SIGNAL_GENERATOR:pcb-library/3D Models/TL2230.STEP"
+    (model "${SIGNAL_GENERATOR}/3D Models/TL2230.STEP"
       (offset (xyz 3.5 -3.5 0))
       (scale (xyz 1 1 1))
@@
     )
   )
-  (footprint "Connector_PinHeader_2.54mm:PinHeader_1x04_P2.54mm_Vertical" (layer "B.Cu")
-    (at 124.04 107.5 90)
-    (descr "Through hole straight pin header, 1x04, 2.54mm pitch, single row")
-    (tags "Through hole pin header THT 1x04 2.54mm single row")
-    (property "Sheetfile" "MCU.kicad_sch")
-    (property "Sheetname" "MCU")
-    (property "ki_description" "Generic connector, single row, 01x04, script generated (kicad-library-utils/schlib/autogen/connector/)")
-    (property "ki_keywords" "connector")
-    (attr through_hole)
-    (fp_text reference "J6" (at 0 2.33 270) (layer "B.SilkS") hide
-        (effects (font (size 1 1) (thickness 0.15)) (justify mirror))
-    )
-    (fp_text value "Conn_01x04" (at 0 -9.95 270) (layer "B.Fab") hide
-        (effects (font (size 1 1) (thickness 0.15)) (justify mirror))
-    )
-    (fp_text user "${REFERENCE}" (at 0 -3.81) (layer "B.Fab")
-        (effects (font (size 1 1) (thickness 0.15)) (justify mirror))
-    )
-    (fp_line (start -1.33 -8.95) (end 1.33 -8.95)
-      (stroke (width 0.12) (type solid)) (layer "B.SilkS"))
-    (fp_line (start -1.33 -1.27) (end -1.33 -8.95)
-      (stroke (width 0.12) (type solid)) (layer "B.SilkS"))
-    (fp_line (start -1.33 -1.27) (end 1.33 -1.27)
-      (stroke (width 0.12) (type solid)) (layer "B.SilkS"))
-    (fp_line (start -1.33 0) (end -1.33 1.33)
-      (stroke (width 0.12) (type solid)) (layer "B.SilkS"))
-    (fp_line (start -1.33 1.33) (end 0 1.33)
-      (stroke (width 0.12) (type solid)) (layer "B.SilkS"))
-    (fp_line (start 1.33 -1.27) (end 1.33 -8.95)
-      (stroke (width 0.12) (type solid)) (layer "B.SilkS"))
-    (fp_line (start -1.8 -9.4) (end 1.8 -9.4)
-      (stroke (width 0.05) (type solid)) (layer "B.CrtYd"))
-    (fp_line (start -1.8 1.8) (end -1.8 -9.4)
-      (stroke (width 0.05) (type solid)) (layer "B.CrtYd"))
-    (fp_line (start 1.8 -9.4) (end 1.8 1.8)
-      (stroke (width 0.05) (type solid)) (layer "B.CrtYd"))
-    (fp_line (start 1.8 1.8) (end -1.8 1.8)
-      (stroke (width 0.05) (type solid)) (layer "B.CrtYd"))
-    (fp_line (start -1.27 -8.89) (end -1.27 0.635)
-      (stroke (width 0.1) (type solid)) (layer "B.Fab"))
-    (fp_line (start -1.27 0.635) (end -0.635 1.27)
-      (stroke (width 0.1) (type solid)) (layer "B.Fab"))
-    (fp_line (start -0.635 1.27) (end 1.27 1.27)
-      (stroke (width 0.1) (type solid)) (layer "B.Fab"))
-    (fp_line (start 1.27 -8.89) (end -1.27 -8.89)
-      (stroke (width 0.1) (type solid)) (layer "B.Fab"))
-    (fp_line (start 1.27 1.27) (end 1.27 -8.89)
-      (stroke (width 0.1) (type solid)) (layer "B.Fab"))
-    (pad "1" thru_hole rect (at 0 0 90) (size 1.7 1.7) (drill 1) (layers "*.Cu" "*.Mask")
-      (net 59 "/MCU/NRST") (pinfunction "Pin_1") (pintype "passive"))
-    (pad "2" thru_hole oval (at 0 -2.54 90) (size 1.7 1.7) (drill 1) (layers "*.Cu" "*.Mask")
-      (net 46 "/MCU/SWDIO") (pinfunction "Pin_2") (pintype "passive"))
-    (pad "3" thru_hole oval (at 0 -5.08 90) (size 1.7 1.7) (drill 1) (layers "*.Cu" "*.Mask")
-      (net 37 "/MCU/SWCLK") (pinfunction "Pin_3") (pintype "passive"))
-    (pad "4" thru_hole oval (at 0 -7.62 90) (size 1.7 1.7) (drill 1) (layers "*.Cu" "*.Mask")
-      (net 3 "GND") (pinfunction "Pin_4") (pintype "passive"))
-    (model "${KICAD6_3DMODEL_DIR}/Connector_PinHeader_2.54mm.3dshapes/PinHeader_1x04_P2.54mm_Vertical.wrl"
-      (offset (xyz 0 0 0))
-      (scale (xyz 1 1 1))
-      (rotate (xyz 0 0 0))
-    )
-  )
   (footprint "Signal Generator Components:MEM2080-00-128-00-A" (layer "B.Cu")
     (at 97.015 127.18 -90)
@@
       )
     )
-    (model ":SIGNAL_GENERATOR:pcb-library/3D Models/MEM2080-00-128-00-A.step"
+    (model "${SIGNAL_GENERATOR}/3D Models/MEM2080-00-128-00-A.step"
       (offset (xyz 7.875 7 0))
       (scale (xyz 1 1 1))
